File: Lab2.sch (KiCad schematic (older format))
At the start: 43 parts, among them SW1 notS, SW2 notR, U1A 7408, U1A? 7408, U1B 7404, U1B? 7404, U2A 7408, U2B 7404, U2B? 7404

Commit message: Changed references to gates
Parts:
- D0, D1, D2, D3, D4, D5, D6, D7, D_CLK: value LED_ALT -> LED
- gave numbers to parts that had none: 17
- renumbered U1A to U3A, U2A to U4A
Connections:
- net GND: now also D0.1 (K), D1.1 (K), D2.1 (K), D3.1 (K), D4.1 (K), D5.1 (K), D6.1 (K), D7.1 (K), D_CLK.1 (K)
Other:
- moved on the sheet: D0, D1, D2, D3, D4, D5, D6, D7, D_CLK
